Commit message: final mapping optimization

File: src/jackal_description/urdf/accessories.urdf.xacro (robot description, xacro)
@@ -176,7 +176,22 @@
     <xacro:property name="parent" value="$(optenv JACKAL_LASER_3D_PARENT ${mount}_mount)" />
     <xacro:property name="lidar_3d_model" value="$(optenv JACKAL_LASER_3D_MODEL vlp16)" />
+    <xacro:property name="lidar_3d_hz" value="$(optenv JACKAL_LASER_3D_HZ 10)" />
+    <xacro:property name="lidar_3d_gpu" value="$(optenv JACKAL_LASER_3D_GPU false)" />
+    <xacro:property name="lidar_3d_organize_cloud" value="$(optenv JACKAL_LASER_3D_ORGANIZE_CLOUD false)" />
+    <xacro:property name="lidar_3d_samples" value="$(optenv JACKAL_LASER_3D_SAMPLES 1875)" />
+    <xacro:property name="lidar_3d_min_angle" value="$(optenv JACKAL_LASER_3D_MIN_ANGLE -3.1415926535897931)" />
+    <xacro:property name="lidar_3d_max_angle" value="$(optenv JACKAL_LASER_3D_MAX_ANGLE 3.1415926535897931)" />
     <!-- Velodyne VLP16 -->
     <xacro:if value="${lidar_3d_model == 'vlp16'}">
-      <xacro:vlp16_mount topic="${topic}" tower="${tower}" prefix="${prefix}" parent_link="${parent}" >
+      <xacro:vlp16_mount topic="${topic}"
+                         tower="${tower}"
+                         prefix="${prefix}"
+                         parent_link="${parent}"
+                         hz="${lidar_3d_hz}"
+                         gpu="${lidar_3d_gpu}"
+                         organize_cloud="${lidar_3d_organize_cloud}"
+                         samples="${lidar_3d_samples}"
+                         min_angle="${lidar_3d_min_angle}"
+                         max_angle="${lidar_3d_max_angle}">
         <origin xyz="$(optenv JACKAL_LASER_3D_OFFSET 0 0 0)" rpy="$(optenv JACKAL_LASER_3D_RPY 0 0 0)" />
       </xacro:vlp16_mount>

File: src/jackal_description/urdf/accessories/vlp16_mount.urdf.xacro (robot description, xacro)
@@ -1,5 +1,5 @@
 <robot xmlns:xacro="http://wiki.ros.org/xacro">
   <xacro:include filename="$(find velodyne_description)/urdf/VLP-16.urdf.xacro" />
-  <xacro:macro name="vlp16_mount" params="prefix parent_link topic tower height:=0.1 *origin">
+  <xacro:macro name="vlp16_mount" params="prefix parent_link topic tower height:=0.1 hz:=10 gpu:=false organize_cloud:=false samples:=1875 min_angle:=-3.1415926535897931 max_angle:=3.1415926535897931 *origin">
     <xacro:if value="${tower}">
       <link name="${prefix}_vlp16_mount" />
@@ -87,10 +87,24 @@
         <origin xyz="0 0 ${height}" rpy="0 0 0" />
       </joint>
-      <xacro:VLP-16 parent="${prefix}_vlp16_plate" topic="${topic}">
+      <xacro:VLP-16 parent="${prefix}_vlp16_plate"
+                    topic="${topic}"
+                    hz="${hz}"
+                    gpu="${gpu}"
+                    organize_cloud="${organize_cloud}"
+                    samples="${samples}"
+                    min_angle="${min_angle}"
+                    max_angle="${max_angle}">
         <origin xyz="0 0 0" rpy="0 0 0" />
       </xacro:VLP-16>
     </xacro:if>
     <xacro:unless value="${tower}">
-      <xacro:VLP-16 parent="${parent_link}" topic="${topic}">
+      <xacro:VLP-16 parent="${parent_link}"
+                    topic="${topic}"
+                    hz="${hz}"
+                    gpu="${gpu}"
+                    organize_cloud="${organize_cloud}"
+                    samples="${samples}"
+                    min_angle="${min_angle}"
+                    max_angle="${max_angle}">
         <xacro:insert_block name="origin" />
       </xacro:VLP-16>
